File: latest.sch (KiCad schematic (older format))
At the start: 41 parts, among them IC1 BA4580R, IC2 BA4580R, IC3 BA4580R, X1 BARREL_JACK, X2 JACK_2P, X3 JACK_2P, X4 JACK_2P, X5 JACK_2P, X6 JACK_2P

Commit message: yay
Parts:
- removed C10, C11, C12: 20p, symbol C
- removed C4, C5, C6: 1uf, symbol CP
- removed IC3: BA4580R, symbol BA4580R
- removed R12, R13, R14: 4k7, symbol R
- removed R5, R6, R7: 10k, symbol R
- removed VR2, VR3, VR4: POT, symbol POT
- removed X3, X4, X5: JACK_2P, symbol JACK_2P
- added C? (x4): 20p, symbol C
- added C? (x4): 1uf, symbol CP
- added IC?: BA4580R, symbol BA4580R
- added R? (x4): 4k7, symbol R
- added R? (x4): 10k, symbol R
- added VR? (x4): POT, symbol POT
- added X? (x4): JACK_2P, symbol JACK_2P
- renumbered R9 to R8, R8 to R9
Connections:
- net labels added: vcc
- wire segments 79 -> 80
Other:
- moved on the sheet: C1, C2, C3, C7, C8, C9, D1, IC1A, IC2A, LD1, R1, R10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

Commit message: yay
Parts:
- gave numbers to parts that had none: 18
Connections:
- wire segments 80 -> 77
Changed lines of the file:
@@
 Connection ~ 5650 6350
 Wire Wire Line
-	9600 5150 9600 4850
-Wire Wire Line
-	9600 4850 9750 4850
-Connection ~ 9750 4850
-Wire Wire Line
-	9750 5050 9550 5050
+	9550 5050 9750 5050
 $Comp
 L C C?
@@
 	14850 5650 14650 5650
 $Comp
-L C C?
+L C C10
 U 1 1 57181077
 P 7750 4850
-F 0 "C?" H 7775 4950 50  0000 L CNN
+F 0 "C10" H 7775 4950 50  0000 L CNN
 F 1 "20p" H 7775 4750 50  0000 L CNN
 F 2 "" H 7788 4700 50  0000 C CNN
@@
 $EndComp
 $Comp
-L R R?
+L R R12
 U 1 1 5718107D
 P 7100 4750
-F 0 "R?" V 7180 4750 50  0000 C CNN
+F 0 "R12" V 7180 4750 50  0000 C CNN
 F 1 "4k7" V 7100 4750 50  0000 C CNN
 F 2 "" V 7030 4750 50  0000 C CNN
@@
 $EndComp
 $Comp
-L POT VR?
+L POT VR2
 U 1 1 57181083
 P 7400 4900
-F 0 "VR?" H 7400 4820 50  0000 C CNN
+F 0 "VR2" H 7400 4820 50  0000 C CNN
 F 1 "POT" H 7400 4900 50  0000 C CNN
 F 2 "" H 7400 4900 50  0000 C CNN
@@
 $EndComp
 $Comp
-L CP C?
+L CP C3
 U 1 1 57181089
 P 7100 4450
-F 0 "C?" H 7125 4550 50  0000 L CNN
+F 0 "C3" H 7125 4550 50  0000 L CNN
 F 1 "1uf" H 7125 4350 50  0000 L CNN
 F 2 "" H 7138 4300 50  0000 C CNN
@@
 $EndComp
 $Comp
-L JACK_2P X?
+L JACK_2P X3
 U 1 1 5718108F
 P 7200 3850
-F 0 "X?" H 6850 3650 50  0000 C CNN
+F 0 "X3" H 6850 3650 50  0000 C CNN
 F 1 "JACK_2P" H 7050 4100 50  0000 C CNN
 F 2 "" H 7200 3850 50  0000 C CNN
@@
 $EndComp
 $Comp
-L R R?
+L R R5
 U 1 1 57181096
 P 7850 4150
-F 0 "R?" V 7930 4150 50  0000 C CNN
+F 0 "R5" V 7930 4150 50  0000 C CNN
 F 1 "10k" V 7850 4150 50  0000 C CNN
 F 2 "" V 7780 4150 50  0000 C CNN
@@
 $EndComp
 $Comp
-L C C?
+L C C11
 U 1 1 5718223D
 P 5700 5300
-F 0 "C?" H 5725 5400 50  0000 L CNN
+F 0 "C11" H 5725 5400 50  0000 L CNN
 F 1 "20p" H 5725 5200 50  0000 L CNN
 F 2 "" H 5738 5150 50  0000 C CNN
@@
 $EndComp
 $Comp
-L R R?
+L R R13
 U 1 1 57182243
 P 6450 5300
-F 0 "R?" V 6530 5300 50  0000 C CNN
+F 0 "R13" V 6530 5300 50  0000 C CNN
 F 1 "4k7" V 6450 5300 50  0000 C CNN
 F 2 "" V 6380 5300 50  0000 C CNN
@@
 $EndComp
 $Comp
-L POT VR?
+L POT VR3
 U 1 1 57182249
 P 6050 5450
-F 0 "VR?" H 6050 5370 50  0000 C CNN
+F 0 "VR3" H 6050 5370 50  0000 C CNN
 F 1 "POT" H 6050 5450 50  0000 C CNN
 F 2 "" H 6050 5450 50  0000 C CNN
@@
 $EndComp
 $Comp
-L CP C?
+L CP C5
 U 1 1 5718224F
 P 6450 4800
-F 0 "C?" H 6475 4900 50  0000 L CNN
+F 0 "C5" H 6475 4900 50  0000 L CNN
 F 1 "1uf" H 6475 4700 50  0000 L CNN
 F 2 "" H 6488 4650 50  0000 C CNN
@@
 $EndComp
 $Comp
-L JACK_2P X?
+L JACK_2P X4
 U 1 1 57182255
 P 6350 3850
-F 0 "X?" H 6000 3650 50  0000 C CNN
+F 0 "X4" H 6000 3650 50  0000 C CNN
 F 1 "JACK_2P" H 6200 4100 50  0000 C CNN
 F 2 "" H 6350 3850 50  0000 C CNN
@@
 VCC
 $Comp
-L R R?
+L R R6
 U 1 1 5718225C
 P 5850 4200
-F 0 "R?" V 5930 4200 50  0000 C CNN
+F 0 "R6" V 5930 4200 50  0000 C CNN
 F 1 "10k" V 5850 4200 50  0000 C CNN
 F 2 "" V 5780 4200 50  0000 C CNN
@@
 	5650 6350 5650 5950
 Wire Wire Line
-	5700 5150 5700 4850
-Wire Wire Line
-	5700 4850 5850 4850
-Connection ~ 5850 4850
-Wire Wire Line
-	5850 5050 5650 5050
-$Comp
-L C C?
+	5650 5050 5850 5050
+$Comp
+L C C12
 U 1 1 5718227D
 P 3850 4850
-F 0 "C?" H 3875 4950 50  0000 L CNN
+F 0 "C12" H 3875 4950 50  0000 L CNN
 F 1 "20p" H 3875 4750 50  0000 L CNN
 F 2 "" H 3888 4700 50  0000 C CNN
@@
 $EndComp
 $Comp
-L R R?
+L R R14
 U 1 1 57182283
 P 3200 4750
-F 0 "R?" V 3280 4750 50  0000 C CNN
+F 0 "R14" V 3280 4750 50  0000 C CNN
 F 1 "4k7" V 3200 4750 50  0000 C CNN
 F 2 "" V 3130 4750 50  0000 C CNN
@@
 $EndComp
 $Comp
-L POT VR?
+L POT VR4
 U 1 1 57182289
 P 3500 4900
-F 0 "VR?" H 3500 4820 50  0000 C CNN
+F 0 "VR4" H 3500 4820 50  0000 C CNN
 F 1 "POT" H 3500 4900 50  0000 C CNN
 F 2 "" H 3500 4900 50  0000 C CNN
@@
 $EndComp
 $Comp
-L CP C?
+L CP C6
 U 1 1 5718228F
 P 3200 4450
-F 0 "C?" H 3225 4550 50  0000 L CNN
+F 0 "C6" H 3225 4550 50  0000 L CNN
 F 1 "1uf" H 3225 4350 50  0000 L CNN
 F 2 "" H 3238 4300 50  0000 C CNN
@@
 $EndComp
 $Comp
-L JACK_2P X?
+L JACK_2P X5
 U 1 1 57182295
 P 3300 3850
-F 0 "X?" H 2950 3650 50  0000 C CNN
+F 0 "X5" H 2950 3650 50  0000 C CNN
 F 1 "JACK_2P" H 3150 4100 50  0000 C CNN
 F 2 "" H 3300 3850 50  0000 C CNN
@@
 $EndComp
 $Comp
-L R R?
+L R R7
 U 1 1 5718229B
 P 3950 4150
-F 0 "R?" V 4030 4150 50  0000 C CNN
+F 0 "R7" V 4030 4150 50  0000 C CNN
 F 1 "10k" V 3950 4150 50  0000 C CNN
 F 2 "" V 3880 4150 50  0000 C CNN
@@
 Wire Wire Line
 	3950 3200 3950 4000
-Wire Wire Line
-	3950 4300 3950 4650
 Connection ~ 3950 4650
 Wire Wire Line
-	3850 4700 3850 4500
-Wire Wire Line
-	3850 4500 3950 4500
-Connection ~ 3950 4500
-Wire Wire Line
 	800  5600 4050 5600
+Connection ~ 9750 3200
+Connection ~ 2900 1350
+Connection ~ 1100 1900
+Wire Wire Line
+	9600 5150 9600 5050
+Connection ~ 9600 5050
+Wire Wire Line
+	5700 5150 5700 5050
+Connection ~ 5700 5050
+Wire Wire Line
+	3850 4700 3850 4650
+Connection ~ 3850 4650
+Wire Wire Line
+	3950 4650 3950 4300
+Text Label 2700 1900 0    60   ~ 0
+VCC
 $EndSCHEMATC
