File: nextest.sch (KiCad schematic (older format))
At the start: 50 parts, among them IC1 BA4580R, IC2 BA4580R, J1 JACK_TRS_6PINS, J2 JACK_TRS_6PINS, J3 JACK_TRS_6PINS, X1 BARREL_JACK

Commit message: thurs2
Parts:
- added J?: JACK_TRS_6PINS, symbol JACK_TRS_6PINS
- added R? (x2): 1k, symbol R
- added R? (x4): 15k, symbol R
- added RV?: 10k, symbol POT
Connections:
- net labels added: INPUT_2
- net labels removed: INPUT_2_is_identical
- wire segments 81 -> 96
Other:
- moved on the sheet: C1, C10, C11, C12, C13, C14, C5, C6, C7, C8, C9, D1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

Commit message: thurs3
Parts:
- added C? (x6): 20p, symbol C
- added C? (x4): 1uf, symbol CP
- added C? (x2): 47uf, symbol CP1
- added IC? (x3): BA4580R, symbol BA4580R
- added R? (x6): 4k7, symbol R
- added R? (x4): 10k, symbol R
- added R? (x2): 47, symbol R
- added RV?: DUAL_POT, symbol DUAL_POT
- added VR? (x4): POT, symbol POT
Connections:
- net labels added: MASTER, POWER, V_EARTH
- wire segments 96 -> 151
Other:
- moved on the sheet: C1, C2, C3, C4, C5, C6, D1, IC1A, LD1, R1, R2, R3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
