File: nextest.sch (KiCad schematic (older format))
At the start: 90 parts, among them IC1 BA4580R, IC2 BA4580R, J1 JACK_TRS_6PINS, J2 JACK_TRS_6PINS, J3 JACK_TRS_6PINS, X1 BARREL_JACK

Commit message: friday
Parts:
- gave numbers to parts that had none: 39
- renumbered C1 to C13, C2 to C14, C3 to C15, C4 to C16, C7 to C17, C8 to C18, C9 to C19, C10 to C20, C11 to C21, C12 to C22, C13 to C23, C14 to C24, C5 to C25, C6 to C26, IC1 to IC2, IC2 to IC3, IC1 to IC3, J3 to J4, R1 to R13, R2 to R14, R3 to R15, R4 to R16, R11 to R17, R12 to R18, R9 to R19, R10 to R20, R13 to R21, R14 to R22, R15 to R23, R16 to R24, R17 to R31, R18 to R32, R19 to R33, R20 to R34, R21 to R35, R22 to R36, R5 to R37, R6 to R38, R7 to R39, R8 to R40, RV1 to RV2, RV2 to RV4, VR1 to VR5, VR2 to VR6, VR3 to VR7, VR4 to VR8
Connections:
- net labels removed: BAL, INPUT_1, INPUT_2, INPUT_3/4, MASTER, OUTPUT_L/R, PAN, POWER, SUM_TO_MONO, V_EARTH
- wire segments 151 -> 191
Other:
- note added: "BAL"
- note added: "INPUT 1\n"
- note added: "INPUT 2\n"
- note added: "INPUT 3/4\n"
- note added: "MASTER\n"
- note added: "OUTPUT L/R"
- note added: "PAN\n"
- note added: "POWER"
- note added: "SUM TO MONO\n"
- note added: "V EARTH"
