File: again.sch (KiCad schematic (older format))
At the start: 62 parts, among them IC2 BA4580R, IC3 BA4580R, J1 JACK_TRS_6PINS, J2 JACK_TRS_6PINS, J3 JACK_TRS_6PINS, J4 JACK_TRS_6PINS, X1 BARREL_JACK

Commit message: friday2
Connections:
- wire segments 94 -> 113
Other:
- note added: "LAMP\n\n"
- note added: "MASTER\nVOLUME"
- note added: "ST BAL"
- note added: "V EARTH\n"
- note removed: "BAL"
- note removed: "MASTER\n"
- moved on the sheet: C17, C18, C21, C22, C25, LD1, R17, R18, R19, R23, R24, R33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

Commit message: monday
Connections:
- wire segments 113 -> 90
Changed lines of the file:
@@
 	3000 4850 3250 4850
 Wire Wire Line
-	3000 5100 3000 5150
-Wire Wire Line
-	3000 5150 3000 5800
-Wire Wire Line
-	3000 3700 3000 4600
-Wire Wire Line
-	3000 4600 3000 4850
-Wire Wire Line
-	2800 5150 3000 5150
-Wire Wire Line
-	3000 5150 3250 5150
+	3000 5100 3000 5800
+Wire Wire Line
+	3000 3700 3000 4850
+Wire Wire Line
+	2800 5150 3250 5150
 $Comp
 L R R14
@@
 Connection ~ 1000 4200
 Wire Wire Line
-	750  4200 1000 4200
-Wire Wire Line
-	1000 4200 1200 4200
-Wire Wire Line
-	750  4600 1000 4600
-Wire Wire Line
-	1000 4600 1200 4600
-Wire Wire Line
-	1000 3700 1000 4200
-Wire Wire Line
-	1000 4200 1000 4300
+	750  4200 1200 4200
+Wire Wire Line
+	750  4600 1200 4600
+Wire Wire Line
+	1000 3700 1000 4300
 Connection ~ 1000 4600
 $Comp
@@
 $EndComp
 Wire Wire Line
-	8950 3450 8950 3850
-Wire Wire Line
-	8950 3850 8950 4300
+	8950 3450 8950 4300
 Connection ~ 8950 3850
 Wire Wire Line
@@
 Connection ~ 8800 3300
 Wire Wire Line
-	8750 3850 8800 3850
-Wire Wire Line
-	8800 3850 8950 3850
+	8750 3850 8950 3850
 $Comp
 L C C22
@@
 Connection ~ 7050 3850
 Wire Wire Line
-	6900 4250 7050 4250
-Wire Wire Line
-	7050 4250 7150 4250
+	6900 4250 7150 4250
 Connection ~ 7050 4250
 Wire Wire Line
@@
 Wire Wire Line
 	6900 3700 6900 3250
-Wire Wire Line
-	6900 2550 7750 2550
 Wire Wire Line
 	7850 2550 8950 2550
@@
 Connection ~ 10450 2500
 Wire Wire Line
-	10900 1800 10900 2200
-Wire Wire Line
-	10150 2500 10450 2500
-Wire Wire Line
-	10450 2500 10900 2500
+	10900 1800 10900 2650
+Wire Wire Line
+	10150 2500 10900 2500
 Wire Wire Line
 	10900 2200 10450 2200
@@
 $EndComp
 Wire Wire Line
-	6150 3450 6150 3850
-Wire Wire Line
-	6150 3850 6150 4250
+	6150 3450 6150 4250
 Connection ~ 6150 3850
 Wire Wire Line
@@
 Connection ~ 6000 3300
 Wire Wire Line
-	5950 3850 6000 3850
-Wire Wire Line
-	6000 3850 6150 3850
+	5950 3850 6150 3850
 $Comp
 L C C18
@@
 Connection ~ 4250 3850
 Wire Wire Line
-	4100 4250 4250 4250
-Wire Wire Line
-	4250 4250 4350 4250
+	4100 4250 4350 4250
 Connection ~ 4250 4250
 Wire Wire Line
@@
 $EndComp
 Wire Wire Line
-	4400 2300 4500 2300
-Wire Wire Line
-	4500 2300 4600 2300
+	4400 2300 4600 2300
 $Comp
 L R R17
@@
 $EndComp
 Wire Wire Line
-	4050 4650 4250 4650
-Wire Wire Line
-	4250 4650 4750 4650
-Wire Wire Line
-	4050 4950 4050 5100
-Wire Wire Line
-	4050 5100 4050 5300
-Wire Wire Line
-	4750 4950 4750 5100
-Wire Wire Line
-	4750 5100 4750 5300
+	4050 4650 4750 4650
+Wire Wire Line
+	4050 4950 4050 5300
+Wire Wire Line
+	4750 4950 4750 5300
 Wire Wire Line
 	4550 5100 4750 5100
@@
 	7850 5050 7850 4950
 Wire Wire Line
-	7850 4950 7950 4950
-Wire Wire Line
-	7950 4950 8050 4950
+	7850 4950 8050 4950
 Wire Wire Line
 	8050 4950 8050 5050
@@
 $EndComp
 Wire Wire Line
-	5550 2300 5650 2300
-Wire Wire Line
-	5650 2300 5750 2300
+	5550 2300 5750 2300
 Wire Wire Line
 	4100 2400 4600 2400
@@
 $EndComp
 Wire Wire Line
-	5400 4650 5750 4650
-Wire Wire Line
-	5750 4650 6100 4650
-Wire Wire Line
-	5400 4950 5400 5100
-Wire Wire Line
-	5400 5100 5400 5300
-Wire Wire Line
-	6100 4950 6100 5100
-Wire Wire Line
-	6100 5100 6100 5300
+	5400 4650 6100 4650
+Wire Wire Line
+	5400 4950 5400 5300
+Wire Wire Line
+	6100 4950 6100 5300
 Wire Wire Line
 	5900 5100 6100 5100
@@
 	7950 4950 7950 4800
 Wire Wire Line
-	10900 2650 10900 2150
+	10900 2200 10900 2150
 Text GLabel 5750 5400 3    60   Input ~ 0
 VE
@@
 	9600 2900 9600 3250
 Wire Wire Line
-	10150 2500 10150 2900
-Wire Wire Line
-	10150 2900 10150 3250
+	10150 2500 10150 3250
 Wire Wire Line
 	10000 2900 10150 2900
@@
 Text Notes 9400 3650 0    60   ~ 0
 V EARTH\n
+Wire Wire Line
+	7650 2550 6900 2550
 $EndSCHEMATC

Commit message: monday2
Parts:
- gave numbers to parts that had none: 2
- renumbered C13 to C1, C22 to C10, C23 to C11, C24 to C12, C25 to C13, C26 to C14, C14 to C2, C15 to C3, C16 to C4, C17 to C5, C18 to C6, C19 to C7, C20 to C8, C21 to C9, IC2 to IC1, IC3 to IC1, IC3 to IC2, R13 to R1, R22 to R10, R23 to R11, R24 to R12, R25 to R13, R26 to R14, R27 to R15, R28 to R16, R29 to R17, R30 to R18, R31 to R19, R14 to R2, R32 to R20, R33 to R21, R34 to R22, R35 to R25, R36 to R26, R37 to R27, R38 to R28, R39 to R29, R15 to R3, R40 to R30, R16 to R4, R17 to R5, R18 to R6, R19 to R7, R20 to R8, R21 to R9, VR5 to VR1, VR6 to VR2, VR7 to VR3, VR8 to VR4
Other:
- moved on the sheet: C13, R27, R28
